Commit message: improved slam

File: ebot_description/models/ebot/ebot_description.xacro (robot description, xacro)
@@ -40,5 +40,5 @@
     <parent link="ebot_base_link" />
     <child link="ebot_base" />
-    <origin xyz="0.0 0.0 0.0" rpy="0.0 0.0 0.0" />
+    <origin xyz="0.2 0.0 0.0" rpy="0.0 0.0 0.0" />
   </joint>
   <link

File: ur_description/urdf/realsense2.urdf.xacro (robot description, xacro)
@@ -79,9 +79,4 @@
             </clip>
           </depth_camera>
-          <noise>
-            <type>gaussian</type>
-            <mean>0.0</mean>
-            <stddev>0.007</stddev>
-          </noise>
         </camera>
         <always_on>1</always_on>
